Commit message: データセットかさ増しプログラム

File: Downuplayer_arm_gnn/merge_joint_robots/merge_baxter.urdf (robot description, URDF)
Before this commit: robot , 20 links, 19 joints
Links:
- link base: mass 97.201099999999997 -> 96.201099999999997; geometry collision mesh filename=../meshes/meshes_baxter/_base.stl; collision sphere radius=0.001
- link head: geometry collision sphere radius=0.001; collision sphere radius=0.001
- link l_gripper_l_finger: geometry collision box size=1.000000000000e-02 1.350000000000e-02 1.127000000000e-01; collision box size=1.000000000000e-02 5.000000000000e-02 1.700000000000e-02
- link l_gripper_r_finger: geometry collision box size=1.000000000000e-02 1.350000000000e-02 1.127000000000e-01; collision box size=1.000000000000e-02 5.000000000000e-02 1.700000000000e-02
- link left_lower_elbow: geometry collision cylinder length=0.10000000000000001 radius=0.059999999999999998; collision cylinder length=0.27200000000000002 radius=0.059999999999999998
- link left_lower_forearm: geometry collision cylinder length=0.10000000000000001 radius=0.059999999999999998; visual mesh filename=../meshes/meshes_baxter/_left_lower_forearm.dae
- link left_lower_shoulder: geometry collision cylinder length=0.12 radius=0.059999999999999998; collision cylinder length=0.27300000000000002 radius=0.059999999999999998
- link left_upper_elbow: geometry collision cylinder length=0.107 radius=0.059999999999999998; visual mesh filename=../meshes/meshes_baxter/_left_upper_elbow.dae
- link left_upper_forearm: geometry collision cylinder length=0.087999999999999995 radius=0.059999999999999998; visual mesh filename=../meshes/meshes_baxter/_left_upper_forearm.dae
- link left_upper_shoulder: geometry collision cylinder length=0.2722 radius=0.059999999999999998; visual mesh filename=../meshes/meshes_baxter/_left_upper_shoulder.dae
- link left_wrist: geometry collision cylinder length=0.046399999999999997 radius=0.040000000000000001; collision cylinder length=0.10000000000000001 radius=0.029000000000000001
- link r_gripper_l_finger: geometry collision box size=1.000000000000e-02 1.350000000000e-02 1.127000000000e-01; collision box size=1.000000000000e-02 5.000000000000e-02 1.700000000000e-02
- link r_gripper_r_finger: geometry collision box size=1.000000000000e-02 1.350000000000e-02 1.127000000000e-01; collision box size=1.000000000000e-02 5.000000000000e-02 1.700000000000e-02
- link right_lower_elbow: geometry collision cylinder length=0.10000000000000001 radius=0.059999999999999998; collision cylinder length=0.27200000000000002 radius=0.059999999999999998
- link right_lower_forearm: geometry collision cylinder length=0.10000000000000001 radius=0.059999999999999998; visual mesh filename=../meshes/meshes_baxter/_right_lower_forearm.dae
- link right_lower_shoulder: geometry collision cylinder length=0.12 radius=0.059999999999999998; collision cylinder length=0.27300000000000002 radius=0.059999999999999998
- link right_upper_elbow: geometry collision cylinder length=0.107 radius=0.059999999999999998; visual mesh filename=../meshes/meshes_baxter/_right_upper_elbow.dae
- link right_upper_forearm: geometry collision cylinder length=0.087999999999999995 radius=0.059999999999999998; visual mesh filename=../meshes/meshes_baxter/_right_upper_forearm.dae
- link right_upper_shoulder: geometry collision cylinder length=0.2722 radius=0.059999999999999998; visual mesh filename=../meshes/meshes_baxter/_right_upper_shoulder.dae
- link right_wrist: geometry collision cylinder length=0.046399999999999997 radius=0.040000000000000001; collision cylinder length=0.10000000000000001 radius=0.029000000000000001
